File: sensor2.sch (KiCad schematic (older format))
At the start: 32 parts, among them CON1 DC2.5-9V, CON2 AVR-ISP-6, CON3 DM3AT-SF-PEJM5, IC1 ATMEGA328P-P, J1 AE-STEREO-MINI, P1 D-SUB9, P2 GMS6-CR6, P3 BATT, Q1 2SC1815, SW1 STOP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

Commit message: Critical miss
Connections:
- net GND: now also SW1.3, SW2.3, SW3.4, SW4.4
- no-connect marks 30 -> 26
Changed lines of the file:
@@
 Sheet 1 1
 Title "sensor2-condor"
-Date "8 sep 2014"
+Date "11 sep 2014"
 Rev "A"
 Comp ""
@@
 $EndComp
 NoConn ~ 8325 6300
-NoConn ~ 7925 6500
-NoConn ~ 9025 6500
 NoConn ~ 9025 6300
-NoConn ~ 9025 5950
 NoConn ~ 9025 5750
-NoConn ~ 7925 5950
 NoConn ~ 8325 5750
 $Comp
@@
 	8475 6500 8475 6650
 Connection ~ 8475 6500
-Connection ~ 9225 6650
-Wire Wire Line
-	8475 6100 9225 6100
-Wire Wire Line
-	8475 6650 9225 6650
-Wire Wire Line
-	9225 6100 9225 6750
 Wire Wire Line
 	8100 1525 8100 5025
@@
 	8625 6300 8400 6300
 Wire Wire Line
-	8400 6300 8400 6100
-Wire Wire Line
-	8400 6100 7675 6100
-Wire Wire Line
-	7675 6100 7675 4500
+	8400 6300 8400 6150
+Wire Wire Line
+	8400 6150 7675 6150
+Wire Wire Line
+	7675 6150 7675 4500
 Wire Wire Line
 	7675 4500 5975 4500
@@
 	8000 3550 8400 3550
 Connection ~ 8400 3550
+Wire Wire Line
+	7925 6500 7925 6650
+Connection ~ 8475 6650
+Wire Wire Line
+	7925 6100 7925 5950
+Connection ~ 8475 6100
+Wire Wire Line
+	9025 5950 9225 5950
+Wire Wire Line
+	9225 5950 9225 6750
+Wire Wire Line
+	7925 6650 9225 6650
+Connection ~ 9225 6650
+Wire Wire Line
+	7925 6100 9225 6100
+Connection ~ 9225 6100
+Wire Wire Line
+	9025 6500 9225 6500
+Connection ~ 9225 6500
 $EndSCHEMATC

Commit message: First release
Connections:
- net GND: no longer P3.2 (PM)
- net at CON1.3: now also P3.2 (PM)
- no-connect marks 26 -> 25
Changed lines of the file:
@@
 Sheet 1 1
 Title "sensor2-condor"
-Date "11 sep 2014"
+Date "12 sep 2014"
 Rev "A"
 Comp ""
@@
 	1875 3775 1650 3775
 Wire Wire Line
-	1650 2950 1650 4425
-Wire Wire Line
 	1650 4075 1400 4075
 Connection ~ 1650 4075
@@
 NoConn ~ 5975 3350
 NoConn ~ 5975 2500
-NoConn ~ 1400 3975
 Connection ~ 3950 3000
 $Comp
@@
 Connection ~ 1550 3150
 Wire Wire Line
-	1650 2950 1200 2950
-Connection ~ 1650 3775
-Wire Wire Line
 	5975 3750 8100 3750
 Connection ~ 8100 3750
@@
 	9025 6500 9225 6500
 Connection ~ 9225 6500
+Wire Wire Line
+	1650 3775 1650 4425
+Wire Wire Line
+	1400 3975 1475 3975
+Wire Wire Line
+	1475 3975 1475 2950
+Wire Wire Line
+	1475 2950 1200 2950
 $EndSCHEMATC

Commit message: Developing
Other:
- moved on the sheet: CON1, P3, U1
Changed lines of the file:
@@
 Sheet 1 1
 Title "sensor2-condor"
-Date "12 sep 2014"
+Date "14 sep 2014"
 Rev "A"
 Comp ""
@@
 L BARREL_JACK CON1
 U 1 1 540BC98C
-P 1100 3975
-F 0 "CON1" H 1100 4225 60  0000 C CNN
-F 1 "DC2.5-9V" H 1100 3775 60  0000 C CNN
-F 2 "" H 1100 3975 60  0000 C CNN
-F 3 "" H 1100 3975 60  0000 C CNN
-	1    1100 3975
+P 925 3975
+F 0 "CON1" H 925 4225 60  0000 C CNN
+F 1 "DC2.5-9V" H 925 3775 60  0000 C CNN
+F 2 "" H 925 3975 60  0000 C CNN
+F 3 "" H 925 3975 60  0000 C CNN
+	1    925  3975
 	1    0    0    -1
 $EndComp
@@
 L SL-TPS63060 U1
 U 1 1 540BC9BB
-P 2425 3975
-F 0 "U1" H 2425 3625 60  0000 C CNN
-F 1 "SL-TPS63060" H 2575 3925 60  0000 C CNN
-F 2 "" H 2175 3975 60  0000 C CNN
-F 3 "" H 2175 3975 60  0000 C CNN
-	1    2425 3975
+P 2750 3975
+F 0 "U1" H 2750 3625 60  0000 C CNN
+F 1 "SL-TPS63060" H 2900 3925 60  0000 C CNN
+F 2 "" H 2500 3975 60  0000 C CNN
+F 3 "" H 2500 3975 60  0000 C CNN
+	1    2750 3975
 	1    0    0    -1
 $EndComp
@@
 	5100 5425 4600 5425
 Wire Wire Line
-	1400 3875 1875 3875
-Wire Wire Line
-	1875 3775 1650 3775
-Wire Wire Line
-	1650 4075 1400 4075
-Connection ~ 1650 4075
+	1225 3875 2200 3875
+Wire Wire Line
+	2200 3775 1975 3775
+Connection ~ 1975 4075
 $Comp
 L +3.3V #PWR017
 U 1 1 540BE159
-P 3350 3550
-F 0 "#PWR017" H 3350 3510 30  0001 C CNN
-F 1 "+3.3V" H 3350 3660 30  0000 C CNN
-F 2 "" H 3350 3550 60  0000 C CNN
-F 3 "" H 3350 3550 60  0000 C CNN
-	1    3350 3550
+P 3600 3550
+F 0 "#PWR017" H 3600 3510 30  0001 C CNN
+F 1 "+3.3V" H 3600 3660 30  0000 C CNN
+F 2 "" H 3600 3550 60  0000 C CNN
+F 3 "" H 3600 3550 60  0000 C CNN
+	1    3600 3550
 	1    0    0    -1
 $EndComp
@@
 L GND #PWR018
 U 1 1 540BE170
-P 3250 4200
-F 0 "#PWR018" H 3250 4200 30  0001 C CNN
-F 1 "GND" H 3250 4130 30  0001 C CNN
-F 2 "" H 3250 4200 60  0000 C CNN
-F 3 "" H 3250 4200 60  0000 C CNN
-	1    3250 4200
-	1    0    0    -1
-$EndComp
-Wire Wire Line
-	3075 3875 3350 3875
-Wire Wire Line
-	3075 3775 3250 3775
+P 3500 4200
+F 0 "#PWR018" H 3500 4200 30  0001 C CNN
+F 1 "GND" H 3500 4130 30  0001 C CNN
+F 2 "" H 3500 4200 60  0000 C CNN
+F 3 "" H 3500 4200 60  0000 C CNN
+	1    3500 4200
+	1    0    0    -1
+$EndComp
+Wire Wire Line
+	3400 3875 3600 3875
+Wire Wire Line
+	3400 3775 3500 3775
 $Comp
 L GND #PWR019
 U 1 1 540BE434
-P 1650 4425
-F 0 "#PWR019" H 1650 4425 30  0001 C CNN
-F 1 "GND" H 1650 4355 30  0001 C CNN
-F 2 "" H 1650 4425 60  0000 C CNN
-F 3 "" H 1650 4425 60  0000 C CNN
-	1    1650 4425
-	1    0    0    -1
-$EndComp
-Wire Wire Line
-	1550 2725 1550 3875
-Connection ~ 1550 3875
+P 1975 4425
+F 0 "#PWR019" H 1975 4425 30  0001 C CNN
+F 1 "GND" H 1975 4355 30  0001 C CNN
+F 2 "" H 1975 4425 60  0000 C CNN
+F 3 "" H 1975 4425 60  0000 C CNN
+	1    1975 4425
+	1    0    0    -1
+$EndComp
 $Comp
 L +BATT #PWR020
 U 1 1 540BE4EF
-P 1550 2725
-F 0 "#PWR020" H 1550 2675 20  0001 C CNN
-F 1 "+BATT" H 1550 2825 30  0000 C CNN
-F 2 "" H 1550 2725 60  0000 C CNN
-F 3 "" H 1550 2725 60  0000 C CNN
-	1    1550 2725
-	1    0    0    -1
-$EndComp
-Wire Wire Line
-	3350 3875 3350 3550
-Wire Wire Line
-	3250 3775 3250 4200
-Wire Wire Line
-	1750 3875 1750 4075
-Wire Wire Line
-	1750 4075 1875 4075
-Connection ~ 1750 3875
-NoConn ~ 1875 4175
-NoConn ~ 1875 3975
-Text Notes 2050 3625 0    60   ~ 0
+P 1575 2725
+F 0 "#PWR020" H 1575 2675 20  0001 C CNN
+F 1 "+BATT" H 1575 2825 30  0000 C CNN
+F 2 "" H 1575 2725 60  0000 C CNN
+F 3 "" H 1575 2725 60  0000 C CNN
+	1    1575 2725
+	1    0    0    -1
+$EndComp
+Wire Wire Line
+	3600 3875 3600 3550
+Wire Wire Line
+	3500 3775 3500 4200
+Wire Wire Line
+	2075 3875 2075 4075
+Wire Wire Line
+	2075 4075 2200 4075
+Connection ~ 2075 3875
+NoConn ~ 2200 4175
+NoConn ~ 2200 3975
+Text Notes 2375 3625 0    60   ~ 0
 EN Jumper ON
 $Comp
@@
 L +3.3V #PWR026
 U 1 1 540BED55
-P 2175 3250
-F 0 "#PWR026" H 2175 3210 30  0001 C CNN
-F 1 "+3.3V" H 2175 3360 30  0000 C CNN
-F 2 "" H 2175 3250 60  0000 C CNN
-F 3 "" H 2175 3250 60  0000 C CNN
-	1    2175 3250
+P 2475 3325
+F 0 "#PWR026" H 2475 3285 30  0001 C CNN
+F 1 "+3.3V" H 2475 3435 30  0000 C CNN
+F 2 "" H 2475 3325 60  0000 C CNN
+F 3 "" H 2475 3325 60  0000 C CNN
+	1    2475 3325
 	1    0    0    -1
 $EndComp
@@
 L VDD #PWR027
 U 1 1 540BED64
-P 2450 3250
-F 0 "#PWR027" H 2450 3350 30  0001 C CNN
-F 1 "VDD" H 2450 3360 30  0000 C CNN
-F 2 "" H 2450 3250 60  0000 C CNN
-F 3 "" H 2450 3250 60  0000 C CNN
-	1    2450 3250
+P 2750 3325
+F 0 "#PWR027" H 2750 3425 30  0001 C CNN
+F 1 "VDD" H 2750 3435 30  0000 C CNN
+F 2 "" H 2750 3325 60  0000 C CNN
+F 3 "" H 2750 3325 60  0000 C CNN
+	1    2750 3325
 	1    0    0    -1
 $EndComp
@@
 L VCC #PWR028
 U 1 1 540BED73
-P 2725 3250
-F 0 "#PWR028" H 2725 3350 30  0001 C CNN
-F 1 "VCC" H 2725 3350 30  0000 C CNN
-F 2 "" H 2725 3250 60  0000 C CNN
-F 3 "" H 2725 3250 60  0000 C CNN
-	1    2725 3250
-	1    0    0    -1
-$EndComp
-Wire Wire Line
-	2725 3375 2725 3250
-Wire Wire Line
-	2175 3375 2725 3375
-Wire Wire Line
-	2175 3375 2175 3250
-Wire Wire Line
-	2450 3250 2450 3375
-Connection ~ 2450 3375
+P 3025 3325
+F 0 "#PWR028" H 3025 3425 30  0001 C CNN
+F 1 "VCC" H 3025 3425 30  0000 C CNN
+F 2 "" H 3025 3325 60  0000 C CNN
+F 3 "" H 3025 3325 60  0000 C CNN
+	1    3025 3325
+	1    0    0    -1
+$EndComp
+Wire Wire Line
+	3025 3450 3025 3325
+Wire Wire Line
+	2475 3450 3025 3450
+Wire Wire Line
+	2475 3450 2475 3325
+Wire Wire Line
+	2750 3325 2750 3450
+Connection ~ 2750 3450
 $Comp
 L PWR_FLAG #FLG029
@@
 L CONN_2 P3
 U 1 1 540BFDBB
-P 850 3050
-F 0 "P3" V 800 3050 40  0000 C CNN
-F 1 "BATT" V 900 3050 40  0000 C CNN
-F 2 "" H 850 3050 60  0000 C CNN
-F 3 "" H 850 3050 60  0000 C CNN
-	1    850  3050
+P 675 3050
+F 0 "P3" V 625 3050 40  0000 C CNN
+F 1 "BATT" V 725 3050 40  0000 C CNN
+F 2 "" H 675 3050 60  0000 C CNN
+F 3 "" H 675 3050 60  0000 C CNN
+	1    675  3050
 	-1   0    0    1
 $EndComp
-Wire Wire Line
-	1200 3150 1550 3150
-Connection ~ 1550 3150
 Wire Wire Line
 	5975 3750 8100 3750
@@
 Connection ~ 9225 6500
 Wire Wire Line
-	1650 3775 1650 4425
-Wire Wire Line
-	1400 3975 1475 3975
-Wire Wire Line
-	1475 3975 1475 2950
-Wire Wire Line
-	1475 2950 1200 2950
+	1975 3775 1975 4425
+Wire Wire Line
+	1225 3975 1425 3975
+Wire Wire Line
+	1425 3975 1425 2950
+Wire Wire Line
+	1425 2950 1025 2950
+Wire Wire Line
+	1975 4075 1225 4075
+Wire Wire Line
+	1025 3150 1575 3150
+Wire Wire Line
+	1575 2725 1575 3875
+Connection ~ 1575 3875
+Connection ~ 1575 3150
 $EndSCHEMATC

Commit message: Connect FSYNC pin to GND
Connections:
- net GND: now also U3.7 (FSYNC)
- no-connect marks 25 -> 24
Changed lines of the file:
@@
 Sheet 1 1
 Title "sensor2-condor"
-Date "14 sep 2014"
+Date "11 feb 2015"
 Rev "A"
 Comp ""
@@
 L GND #PWR09
 U 1 1 540B1794
-P 10850 5000
-F 0 "#PWR09" H 10850 5000 30  0001 C CNN
-F 1 "GND" H 10850 4930 30  0001 C CNN
-F 2 "" H 10850 5000 60  0000 C CNN
-F 3 "" H 10850 5000 60  0000 C CNN
-	1    10850 5000
+P 10850 5450
+F 0 "#PWR09" H 10850 5450 30  0001 C CNN
+F 1 "GND" H 10850 5380 30  0001 C CNN
+F 2 "" H 10850 5450 60  0000 C CNN
+F 3 "" H 10850 5450 60  0000 C CNN
+	1    10850 5450
 	1    0    0    -1
 $EndComp
@@
 NoConn ~ 8625 5225
 NoConn ~ 10525 5225
-NoConn ~ 10525 5125
 $Comp
 L GND #PWR011
@@
 	10525 4825 10850 4825
 Wire Wire Line
-	10850 4825 10850 5000
+	10850 4825 10850 5450
 Wire Wire Line
 	10525 4925 10850 4925
@@
 Connection ~ 1575 3875
 Connection ~ 1575 3150
+Wire Wire Line
+	10525 5125 10850 5125
+Connection ~ 10850 5125
 $EndSCHEMATC
